File: Kicad/tim_keyboard.kicad_sch (KiCad schematic)
At the start: 8 parts, among them J2 RS-232C, J3 TASTATURA, J4 SERIAL, J5 KBD, U8 MC1489, U9 MC1488

Commit message: Fix J4, J5.
Connections:
- net RX0: now also J4.3 (Pin_3)
- net RX1: now also J5.3 (Pin_3)
- net TX0: now also J4.2 (Pin_2)
- net TX1: now also J5.2 (Pin_2)
- net K_RX: no longer names the net of J3.2 (Pin_2), U8.13 (IN_D)
- net K_RX: no longer J5.3 (Pin_3)
- net K_TX: no longer names the net of J3.3 (Pin_3), U9.8 (3Y)
- net K_TX: no longer J5.2 (Pin_2)
- net S_RX: no longer names the net of J2.3, U8.1 (IN_A)
- net S_RX: no longer J4.3 (Pin_3)
- net S_TX: no longer names the net of J2.2, U9.3 (1Y)
- net S_TX: no longer J4.2 (Pin_2)
Changed lines of the file:
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@@
-	)
-	(junction
-		(at 50.8 133.35)
-		(diameter 0)
-		(color 0 0 0 0)
-	)
-	(junction
-		(at 58.42 135.89)
-		(diameter 0)
-		(color 0 0 0 0)
 	)
 	(junction
@@
 	)
 	(junction
-		(at 115.57 78.74)
-		(diameter 0)
-		(color 0 0 0 0)
-	)
-	(junction
-		(at 120.65 96.52)
-		(diameter 0)
-		(color 0 0 0 0)
-	)
-	(junction
 		(at 60.96 165.1)
 		(diameter 0)
@@
 	(wire
 		(pts
-			(xy 120.65 140.97) (xy 120.65 96.52)
+			(xy 120.65 81.28) (xy 120.65 140.97)
+		)
+		(stroke
+			(width 0)
+			(type default)
+		)
+	)
+	(wire
+		(pts
+			(xy 29.21 135.89) (xy 27.94 135.89)
 		)
 		(stroke
@@
 	(wire
 		(pts
+			(xy 134.62 96.52) (xy 135.89 96.52)
+		)
+		(stroke
+			(width 0)
+			(type default)
+		)
+	)
+	(wire
+		(pts
 			(xy 91.44 105.41) (xy 134.62 105.41)
 		)
@@
 	(wire
 		(pts
-			(xy 50.8 133.35) (xy 50.8 171.45)
-		)
-		(stroke
-			(width 0)
-			(type default)
-		)
-	)
-	(wire
-		(pts
-			(xy 27.94 133.35) (xy 50.8 133.35)
+			(xy 50.8 80.01) (xy 50.8 171.45)
 		)
 		(stroke
@@
 	(wire
 		(pts
-			(xy 158.75 78.74) (xy 115.57 78.74)
-		)
-		(stroke
-			(width 0)
-			(type default)
-		)
-	)
-	(wire
-		(pts
 			(xy 97.79 80.01) (xy 50.8 80.01)
 		)
@@
 	(wire
 		(pts
-			(xy 120.65 96.52) (xy 120.65 81.28)
-		)
-		(stroke
-			(width 0)
-			(type default)
-		)
-	)
-	(wire
-		(pts
 			(xy 133.35 46.99) (xy 137.16 46.99)
 		)
@@
 	(wire
 		(pts
-			(xy 135.89 93.98) (xy 115.57 93.98)
+			(xy 135.89 93.98) (xy 134.62 93.98)
 		)
 		(stroke
@@
 	(wire
 		(pts
-			(xy 120.65 96.52) (xy 135.89 96.52)
-		)
-		(stroke
-			(width 0)
-			(type default)
-		)
-	)
-	(wire
-		(pts
 			(xy 100.33 82.55) (xy 54.61 82.55)
 		)
@@
 	(wire
 		(pts
-			(xy 50.8 80.01) (xy 50.8 133.35)
-		)
-		(stroke
-			(width 0)
-			(type default)
-		)
-	)
-	(wire
-		(pts
 			(xy 59.69 38.1) (xy 64.77 38.1)
 		)
@@
 	(wire
 		(pts
-			(xy 58.42 135.89) (xy 58.42 167.64)
+			(xy 58.42 99.06) (xy 58.42 167.64)
 		)
 		(stroke
@@
 	(wire
 		(pts
-			(xy 115.57 93.98) (xy 115.57 78.74)
-		)
-		(stroke
-			(width 0)
-			(type default)
-		)
-	)
-	(wire
-		(pts
 			(xy 129.54 39.37) (xy 137.16 39.37)
 		)
@@
 	(wire
 		(pts
-			(xy 115.57 78.74) (xy 102.87 78.74)
-		)
-		(stroke
-			(width 0)
-			(type default)
-		)
-	)
-	(wire
-		(pts
-			(xy 58.42 99.06) (xy 58.42 135.89)
+			(xy 102.87 78.74) (xy 158.75 78.74)
+		)
+		(stroke
+			(width 0)
+			(type default)
+		)
+	)
+	(wire
+		(pts
+			(xy 29.21 133.35) (xy 27.94 133.35)
 		)
 		(stroke
@@
 	(wire
 		(pts
-			(xy 27.94 135.89) (xy 58.42 135.89)
-		)
-		(stroke
-			(width 0)
-			(type default)
-		)
-	)
-	(wire
-		(pts
 			(xy 43.18 152.4) (xy 81.28 152.4)
 		)
@@
 		)
 	)
-	(label "K_TX"
-		(at 123.19 93.98 0)
-		(fields_autoplaced yes)
-		(effects
-			(font
-				(size 1.27 1.27)
-			)
-			(justify left bottom)
-		)
-	)
-	(label "K_RX"
-		(at 123.19 96.52 0)
-		(fields_autoplaced yes)
-		(effects
-			(font
-				(size 1.27 1.27)
-			)
-			(justify left bottom)
-		)
-	)
-	(label "S_RX"
-		(at 36.83 135.89 0)
-		(fields_autoplaced yes)
-		(effects
-			(font
-				(size 1.27 1.27)
-			)
-			(justify left bottom)
-		)
-	)
-	(label "S_TX"
-		(at 36.83 133.35 0)
-		(fields_autoplaced yes)
-		(effects
-			(font
-				(size 1.27 1.27)
-			)
-			(justify left bottom)
-		)
-	)
 	(global_label "~{RTS0}"
 		(shape input)
@@
 		)
 	)
+	(global_label "TX1"
+		(shape input)
+		(at 134.62 93.98 180)
+		(fields_autoplaced yes)
+		(effects
+			(font
+				(size 1.27 1.27)
+			)
+			(justify right)
+		)
+		(property "Intersheetrefs" "${INTERSHEET_REFS}"
+			(at 128.2482 93.98 0)
+			(effects
+				(font
+					(size 1.27 1.27)
+				)
+				(justify right)
+				(hide yes)
+			)
+		)
+	)
+	(global_label "RX0"
+		(shape input)
+		(at 29.21 135.89 0)
+		(fields_autoplaced yes)
+		(effects
+			(font
+				(size 1.27 1.27)
+			)
+			(justify left)
+		)
+		(property "Intersheetrefs" "${INTERSHEET_REFS}"
+			(at 35.8842 135.89 0)
+			(effects
+				(font
+					(size 1.27 1.27)
+				)
+				(justify left)
+				(hide yes)
+			)
+		)
+	)
+	(global_label "RX1"
+		(shape input)
+		(at 134.62 96.52 180)
+		(fields_autoplaced yes)
+		(effects
+			(font
+				(size 1.27 1.27)
+			)
+			(justify right)
+		)
+		(property "Intersheetrefs" "${INTERSHEET_REFS}"
+			(at 127.9458 96.52 0)
+			(effects
+				(font
+					(size 1.27 1.27)
+				)
+				(justify right)
+				(hide yes)
+			)
+		)
+	)
 	(global_label "~{DCD0}"
 		(shape input)
@@
 				(hide yes)
 			)
+		)
+	)
+	(global_label "TX0"
+		(shape input)
+		(at 29.21 133.35 0)
+		(fields_autoplaced yes)
+		(effects
+			(font
+				(size 1.27 1.27)
+			)
+			(justify left)
+		)
+		(property "Intersheetrefs" "${INTERSHEET_REFS}"
+			(at 35.5818 133.35 0)
+			(effects
+				(font
+					(size 1.27 1.27)
+				)
+				(justify left)
+				(hide yes)
+			)
