File: Kicad/tim_cpu.kicad_sch (KiCad schematic)
At the start: 22 parts, among them T1 RESET, T2 RESET, U14 74LS240, U16 27C128, U17 HD64180, U23 74LS00, U24 74LS04, U7 74LS74, Y1 12.288MHz

Commit message: U18 correction, ROM A13 ground, DB25 mouting hole fix, remove H9, Credits Update
Parts:
- U16: value 27C128 -> 2764
Connections:
- net GND: now also U16.26 (A13)
- no-connect marks 8 -> 7
Changed lines of the file:
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@@
 	)
 	(no_connect
-		(at 76.2 189.23)
-	)
-	(no_connect
 		(at 195.58 196.85)
 	)
@@
 	)
 	(symbol
+		(lib_id "power:GND")
+		(at 76.2 189.23 270)
+		(unit 1)
+		(exclude_from_sim no)
+		(in_bom yes)
+		(on_board yes)
+		(dnp no)
+		(fields_autoplaced yes)
+		(property "Reference" "#PWR0191"
+			(at 69.85 189.23 0)
+			(effects
+				(font
+					(size 1.27 1.27)
+				)
+				(hide yes)
+			)
+		)
+		(property "Value" "GND"
+			(at 72.39 189.2299 90)
+			(effects
+				(font
+					(size 1.27 1.27)
+				)
+				(justify right)
+			)
+		)
+		(property "Footprint" ""
+			(at 76.2 189.23 0)
+			(effects
+				(font
+					(size 1.27 1.27)
+				)
+				(hide yes)
+			)
+		)
+		(property "Datasheet" ""
+			(at 76.2 189.23 0)
+			(effects
+				(font
+					(size 1.27 1.27)
+				)
+				(hide yes)
+			)
+		)
+		(property "Description" "Power symbol creates a global label with name \"GND\" , ground"
+			(at 76.2 189.23 0)
+			(effects
+				(font
+					(size 1.27 1.27)
+				)
+				(hide yes)
+			)
+		)
+		(pin "1"
+		)
+		(instances
+			(project "TIM-011B"
+				(path "/6f8183af-5e43-48c0-9c11-20d9f97fa05a/c54ba189-8dd6-4023-a185-0f00bef03e1c"
+					(reference "#PWR0191")
+					(unit 1)
+				)
+			)
+		)
+	)
+	(symbol
 		(lib_id "Device:C")
 		(at 331.47 57.15 0)
@@
 			)
 		)
-		(property "Value" "27C128"
+		(property "Value" "2764"
 			(at 88.5541 151.13 0)
 			(effects
